Commit message: Change ik solver to tracik.

File: urdf/ur10.urdf (robot description, URDF)
Before this commit: robot robot, 11 links, 10 joints
Links:
- removed link hand
- added link base
- link base_link: geometry 
Joints:
- removed joint tool0-hand
- added joint base_link-base_fixed_joint: type fixed, parent base_link, child base, origin xyz=0 0 0 rpy=0 0 3.14159265359
- joint base_link-base_link_inertia: origin xyz=0 0 0.32 rpy=0 0 3.14159265359 -> xyz=0 0 0.3 rpy=0 0 3.14159265359
- joint flange-tool0: origin xyz=0 0 0 rpy=1.5707963267948966 0 1.5707963267948966 -> xyz=0 0 0 rpy=0 0 3.14159265359
